File: hardware/TCduo/TCduo_v1.brd (EAGLE design)
At the start: 86.8 x 55 mm, 18 parts, among them Q2 600mA/40V, Q3 600mA/40V

Commit message: updated hardware
Parts:
- removed OT1: RED, adafruit:CHIPLED_0805
- removed PAC, PWM: (no value), jumper-piTC2:JP4
- removed Q2, Q3: 600mA/40V, SparkFun-DiscreteSemi:SOT23-3
- removed RN1: EXB-38V102JV, EXB-38V102JV:RESCAXS80P320X160X60-8N
- added J1, J2: JST_6_PIN_VERTICAL, SparkFun-Connectors:JST-6-SMD-VERT-1.0MM
Connections:
- removed net 3V3PWR: ARDUINO_NANO.15, RASPI_GPIO.17
- removed net 5V: RASPI_GPIO.2, RASPI_GPIO.4
- removed net DIO10: ARDUINO_NANO.28, RASPI_GPIO.35, RN1.4
- removed net DIO2: ARDUINO_NANO.20, PAC.3, RASPI_GPIO.15
- removed net DIO9: ARDUINO_NANO.27, RASPI_GPIO.12, RN1.1, RN1.2
- removed net N$1: Q2.1, RN1.5
- removed net N$2: PWM.3
- removed net N$5: Q3.1, RN1.8
- removed net N$6: OT1.A, RN1.7
- new net 3.3V: RASPI_GPIO.17
- new net IO2: ARDUINO_NANO.20, J1.5, J2.5, RASPI_GPIO.15
- net +5V: now also ARDUINO_NANO.15, J1.1, J2.1, RASPI_GPIO.2, RASPI_GPIO.4
- net GND: now also J1.6, J2.6; no longer OT1.C, PAC.2, PWM.2, Q2.2, Q3.2
- net OT1: now also ARDUINO_NANO.27, J1.3, J2.3, RASPI_GPIO.12; no longer PAC.1, PWM.1, Q3.3
- net OT2: now also ARDUINO_NANO.28, J1.4, J2.4, RASPI_GPIO.35; no longer PAC.4, PWM.4, Q2.3
- net VDD: now also J1.2, J2.2
Routing:
- net DIO10: track 140.7 -> 0.00 mm, vias 1 -> 0
- net DIO2: track 140.3 -> 0.00 mm, vias 2 -> 0
- net OT2: track 43.0 -> 173.8 mm, vias 0 -> 1
- net IO2: track 0.00 -> 119.5 mm, vias 0 -> 3
- net +5V: track 21.5 -> 122.2 mm, vias 0 -> 2
- net DIO9: track 80.3 -> 0.00 mm, vias 4 -> 0
- net OT1: track 43.4 -> 115.2 mm, vias 0 -> 6
- net VDD: track 60.5 -> 103.6 mm, vias 0 -> 2
- net 3V3PWR: track 41.0 -> 0.00 mm
- net N$5: track 9.52 -> 0.00 mm
- net +3V3: track 115.4 -> 105.9 mm
- net N$1: track 8.37 -> 0.00 mm
- net N$6: track 6.47 -> 0.00 mm
- net 5V: track 2.54 -> 0.00 mm
- net I2C_DATA: track 132.3 -> 130.9 mm
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Other:
- board text added: "TCduo"
- board text removed: "GND"
- board text removed: "IO2"
- board text removed: "OT1"
- board text removed: "OT2"
- board text removed: "piTC4"
