File: hardware/TCsolo/TCsolo_v1.sch (EAGLE design)
At the start: 18 parts, among them Q2 600mA/40V, Q3 600mA/40V

Commit message: updated hardware
Parts:
- removed CH2: PCC-SMP, PCC-SMP:PCC-SMP
- removed OT1: RED, adafruit:LEDCHIPLED_0805
- removed PAC, PWM: (no value), jumper-piTC2:JP4E
- removed Q2, Q3: 600mA/40V, SparkFun-DiscreteSemi:TRANS_NPN-MMBT2222AL
- removed RASPI_GPIO: RASPBERRYPI-40-PIN-GPIO_PTH, SparkFun-Connectors:RASPBERRYPI-40-PIN-GPIO_PTH
- removed RN1: EXB-38V102JV, EXB-38V102JV:EXB-38V102JV
- added J1, J2: JST_6_PIN_VERTICAL, SparkFun-Connectors:JST_6_PIN_VERTICAL
- added RASPI_IO: (no value), jumper-3:JP6Q
- MCP3422: value MCP3422A0-E/MC -> MCP3422
- renumbered C4 to C3
Connections:
- removed net 3V3PWR: ARDUINO_NANO.VIN, RASPI_GPIO.3.3V@17
- removed net DIO10: ARDUINO_NANO.D10, RASPI_GPIO.GP19, RN1.4
- removed net DIO2: ARDUINO_NANO.D2, PAC.3, RASPI_GPIO.GP22
- removed net DIO9: ARDUINO_NANO.D9, RASPI_GPIO.GP18#, RN1.1, RN1.2
- removed net N$1: Q2.B, RN1.5
- removed net N$2: PWM.3
- removed net N$5: Q3.B, RN1.8
- removed net N$6: OT1.A, RN1.7
- removed net UART_0: ARDUINO_NANO.RX0, RASPI_GPIO.TXO
- removed net UART_1: ARDUINO_NANO.TX1, RASPI_GPIO.RXI
- new net IO2: ARDUINO_NANO.D2, J1.5, J2.5, RASPI_IO.7
- new net SR0: ARDUINO_NANO.RX0, RASPI_IO.8
- new net SR1: ARDUINO_NANO.TX1, RASPI_IO.10
- net +3V3: now also RASPI_IO.1; no longer RASPI_GPIO.3.3V@1
- net +5V: now also ARDUINO_NANO.VIN, J1.1, J2.1, RASPI_IO.2, RASPI_IO.4
- net CH2+: no longer CH2.1
- net CH2-: no longer CH2.2
- net GND: now also J1.6, J2.6, RASPI_IO.6, RASPI_IO.9; no longer OT1.C, PAC.2, PWM.2, Q2.E, Q3.E, RASPI_GPIO.GND@14, RASPI_GPIO.GND@20, RASPI_GPIO.GND@25, RASPI_GPIO.GND@30, RASPI_GPIO.GND@34, RASPI_GPIO.GND@39, RASPI_GPIO.GND@6, RASPI_GPIO.GND@9
- net I2C_CLK: now also RASPI_IO.5; no longer RASPI_GPIO.SCL
- net I2C_DATA: now also RASPI_IO.3; no longer RASPI_GPIO.SDA
- net OT1: now also ARDUINO_NANO.D9, J1.3, J2.3, RASPI_IO.12; no longer PAC.1, PWM.1, Q3.C
- net OT2: now also ARDUINO_NANO.D10, J1.4, J2.4, RASPI_IO.11; no longer PAC.4, PWM.4, Q2.C
- net VDD: now also J1.2, J2.2
